Commit message: feat: Add level silver VTOL drone asset model and C++ flight controller launch sequence

File: src/robot_description/urdf/inspection_robot.urdf.xacro (robot description, xacro)
@@ -1,62 +1,45 @@
 <?xml version="1.0"?>
-<robot name="inspection_robot"
-       xmlns:xacro="http://ros.org/wiki/xacro">
-  <!-- Base -->
+<robot name="standard_vtol" xmlns:xacro="http://ros.org">
+  <!-- ==================== MAIN AIRFRAME (LEVEL SILVER PLANE) ==================== -->
   <link name="base_link">
-    <visual>
-      <geometry>
-        <box size="1.0 0.6 0.3"/>
-      </geometry>
-      <material name="blue">
-        <color rgba="0 0.2 0.8 1"/>
-      </material>
-    </visual>
+    <inertial>
+      <mass value="2.0"/>
+      <origin xyz="0 0 0" rpy="0 0 0"/>
+      <inertia ixx="0.05" ixy="0.0" ixz="0.0" iyy="0.05" iyz="0.0" izz="0.1"/>
+    </inertial>
     <collision>
       <geometry>
-        <box size="1.0 0.6 0.3"/>
+        <box size="0.6 0.8 0.15"/>
       </geometry>
     </collision>
-    <inertial>
-      <mass value="10"/>
-      <inertia
-        ixx="0.1"
-        ixy="0"
-        ixz="0"
-        iyy="0.1"
-        iyz="0"
-        izz="0.1"/>
-    </inertial>
-  </link>
-  <!-- Left wheel -->
-  <link name="left_wheel">
     <visual>
+      <!-- RE-BALANCED AXES MAP TO POSITION PLANE LEVEL AND FACING FORWARD -->
+      <origin xyz="0 0 0.4" rpy="1.5708 0 -1.5708"/>
       <geometry>
-        <cylinder radius="0.15" length="0.1"/>
+        <mesh filename="file:///home/joel/robotics-portfolio/src/robot_description/meshes/x8_wing.dae" scale="0.001 0.001 0.001"/>
       </geometry>
     </visual>
   </link>
-  <joint name="left_wheel_joint"
-         type="continuous">
-    <parent link="base_link"/>
-    <child link="left_wheel"/>
-    <origin xyz="0 0.35 -0.15"
-            rpy="1.5708 0 0"/>
-    <axis xyz="0 1 0"/>
-  </joint>
-  <!-- Right wheel -->
-  <link name="right_wheel">
+  <!-- ==================== METALLIC SILVER FINISH ==================== -->
+  <gazebo reference="base_link">
     <visual>
-      <geometry>
-        <cylinder radius="0.15" length="0.1"/>
-      </geometry>
+      <material>
+        <ambient>0.75 0.75 0.75 1.0</ambient>
+        <diffuse>0.75 0.75 0.75 1.0</diffuse>
+        <specular>0.9 0.9 0.9 1.0</specular>
+        <emissive>0.0 0.0 0.0 1.0</emissive>
+      </material>
     </visual>
-  </link>
-  <joint name="right_wheel_joint"
-         type="continuous">
-    <parent link="base_link"/>
-    <child link="right_wheel"/>
-    <origin xyz="0 -0.35 -0.15"
-            rpy="1.5708 0 0"/>
-    <axis xyz="0 1 0"/>
-  </joint>
+  </gazebo>
+  <!-- ==================== GAZEBO ROS 3D MOVEMENT ENGINE ==================== -->
+  <gazebo>
+    <plugin name="vtol_flight_core" filename="libgazebo_ros_planar_move.so">
+      <command_topic>cmd_vel</command_topic>
+      <odometry_topic>odom</odometry_topic>
+      <odometry_frame>odom</odometry_frame>
+      <odometry_rate>30.0</odometry_rate>
+      <robot_base_frame>base_link</robot_base_frame>
+      <publish_odometry_tf>true</publish_odometry_tf>
+    </plugin>
+  </gazebo>
 </robot>

Commit message: style: Rotate silver jet mesh orientation an additional 45 degrees right for perfect tracking heading

File: src/robot_description/urdf/inspection_robot.urdf.xacro (robot description, xacro)
@@ -14,6 +14,5 @@
     </collision>
     <visual>
-      <!-- RE-BALANCED AXES MAP TO POSITION PLANE LEVEL AND FACING FORWARD -->
-      <origin xyz="0 0 0.4" rpy="1.5708 0 -1.5708"/>
+      <origin xyz="0 0 0.4" rpy="1.5708 0 -3.1416"/>
       <geometry>
         <mesh filename="file:///home/joel/robotics-portfolio/src/robot_description/meshes/x8_wing.dae" scale="0.001 0.001 0.001"/>
@@ -32,13 +31,9 @@
     </visual>
   </gazebo>
-  <!-- ==================== GAZEBO ROS 3D MOVEMENT ENGINE ==================== -->
+  <!-- ==================== MODERN GAZEBO SIM MOVEMENT ENGINE ==================== -->
   <gazebo>
-    <plugin name="vtol_flight_core" filename="libgazebo_ros_planar_move.so">
-      <command_topic>cmd_vel</command_topic>
-      <odometry_topic>odom</odometry_topic>
-      <odometry_frame>odom</odometry_frame>
-      <odometry_rate>30.0</odometry_rate>
+    <!-- The exact flight physics system required for ROS 2 Jazzy & Gazebo Sim -->
+    <plugin filename="gz-sim-velocity-control-system" name="gz::sim::systems::VelocityControl">
       <robot_base_frame>base_link</robot_base_frame>
-      <publish_odometry_tf>true</publish_odometry_tf>
     </plugin>
   </gazebo>

Commit message: feat: Implement relative-frame cooperative tracking swarm with zero-gravity altitude lock

File: src/robot_description/urdf/inspection_robot.urdf.xacro (robot description, xacro)
@@ -14,5 +14,5 @@
     </collision>
     <visual>
-      <origin xyz="0 0 0.4" rpy="1.5708 0 -3.1416"/>
+      <origin xyz="0 0 0.0" rpy="1.5708 0 -3.1416"/>
       <geometry>
         <mesh filename="file:///home/joel/robotics-portfolio/src/robot_description/meshes/x8_wing.dae" scale="0.001 0.001 0.001"/>
@@ -20,5 +20,5 @@
     </visual>
   </link>
-  <!-- ==================== METALLIC SILVER FINISH ==================== -->
+  <!-- ==================== METALLIC SILVER FINISH & GRAVITY LOCK ==================== -->
   <gazebo reference="base_link">
     <visual>
@@ -30,11 +30,19 @@
       </material>
     </visual>
+    <!-- HARDWARE LOCK: Disables gravity so the jet hovers perfectly at its spawn altitude -->
+    <gravity>0</gravity>
   </gazebo>
-  <!-- ==================== MODERN GAZEBO SIM MOVEMENT ENGINE ==================== -->
+  <!-- ==================== WORKING GAZEBO SIM MOVEMENT ENGINE ==================== -->
   <gazebo>
-    <!-- The exact flight physics system required for ROS 2 Jazzy & Gazebo Sim -->
     <plugin filename="gz-sim-velocity-control-system" name="gz::sim::systems::VelocityControl">
       <robot_base_frame>base_link</robot_base_frame>
     </plugin>
   </gazebo>
+  <!-- ==================== LIVE AERIAL TELEMETRY PUBLISHER ==================== -->
+  <gazebo>
+    <plugin filename="gz-sim-odometry-publisher-system" name="gz::sim::systems::OdometryPublisher">
+      <odom_frame>standard_vtol/odometry</odom_frame>
+      <robot_base_frame>base_link</robot_base_frame>
+    </plugin>
+  </gazebo>
 </robot>
